File: PCB/Main Board/obd.sch (KiCad schematic (older format))
At the start: 1 part

Commit message: Added main firmware project and the main board PCB project.
Parts:
- removed U?: STN1110, ~, symbol STN1110
Changed lines of the file:
@@
 LIBS:valves
 LIBS:SeniorDesign
-LIBS:OBD-cache
+LIBS:atmega32u4bb-from_eagle
+LIBS:main-cache
 EELAYER 27 0
 EELAYER END
@@
 Sheet 1 1
 Title ""
-Date "18 jul 2013"
+Date "22 aug 2013"
 Rev ""
 Comp ""
@@
 Comment4 ""
 $EndDescr
-$Comp
-L STN1110 U?
-U 1 1 51E74A68
-P 5600 4050
-F 0 "U?" H 4150 2500 60  0000 C CNN
-F 1 "STN1110" H 6850 2600 60  0000 C CNN
-F 2 "~" H 4400 2250 60  0000 C CNN
-F 3 "~" H 4400 2250 60  0000 C CNN
-	1    5600 4050
-	1    0    0    -1
-$EndComp
 $EndSCHEMATC
