File: src/PCB/Main Board/avr.sch (KiCad schematic (older format))
At the start: 0 parts

Commit message: Updated PCB projects.
Parts:
- added C? (x2): 18pF, ~, symbol C_SMALL
- added C?: 1uF, ~, symbol CP1
- added C? (x2): 100nF, ~, symbol C_SMALL
- added C? (x2): 10nF, ~, symbol C_SMALL
- added C? (x2): 1nF, ~, symbol C_SMALL
- added C?: 10uF, ~, symbol CP1
- added P?: CONN_6, symbol CONN_6
- added R?: 1M, ~, symbol R_US
- added R?: 300k, ~, symbol R_US
- added R?: 125k, ~, symbol R_US
- added R?: 47k, ~, symbol R_US
- added R?: 10k, ~, symbol R_US
- added R?: 100k, ~, symbol R_US
- added U?: ATMEGA32U4, symbol ADAPROG_ATMEGA32U4
- added X?: 16MHz, ~, symbol CRYSTAL
Connections:
- new net: C?.1, U?.16 (XTAL2), X?.2
- new net: C?.1, U?.17 (XTAL1), X?.1
- new net: C?.1, U?.6 (UCAP)
- new net +5V: C?.1, C?.1, C?.1, C?.1, C?.1, C?.1, C?.1, R?.1, R?.1, R?.1, R?.1, R?.1, U?.14 (VCC), U?.2 (UVCC), U?.24 (AVCC), U?.34 (VCC1), U?.44 (AVCC1), U?.7 (VBUS)
- new net GND: C?.2, C?.2, C?.2, C?.2, C?.2, C?.2, C?.2, C?.2, C?.2, C?.2, R?.2, U?.15 (GND), U?.23 (GND1), U?.35 (GND2), U?.43 (GND3), U?.5 (UGND)
- new net SW1: P?.1, R?.2
- new net SW2: P?.2, R?.2
- new net SW3: P?.3, R?.2
- new net SW4: P?.4, R?.2
- new net SW5: P?.5, R?.2
- new net SW_ADC: P?.6, R?.1, U?.41 (PF0(ADC0))
- new net UART_CTS: U?.22 (PD5(XCK/CTS))
- new net UART_RTS: U?.12 (PB7(OC0A/OC1C/RTS))
- new net UART_RX: U?.20 (PD2(INT2/RXD1))
- new net UART_TX: U?.21 (PD3(INT3/TXD1))
