File: src/PCB/Main Board/main.sch (KiCad schematic (older format))
At the start: 7 parts

Commit message: Updated PCB projects.
Parts:
- removed X?: X_XTAL, adaprog-NX5032, symbol X_XTAL
- added C?: 3.3uF, ~, symbol C_SMALL
- added C? (x5): 100nF, ~, symbol C_SMALL
- added C? (x2): 10nF, ~, symbol C_SMALL
- added C? (x2): 1nF, ~, symbol C_SMALL
- added C? (x2): 4.7uF, ~, symbol CP1
- added C?: 3.3uF, ~, symbol CP1
- added D? (x2): RxD, ~, symbol LED
- added D? (x2): TxD, ~, symbol LED
- added FB? (x2): 800mA, ~, symbol FILTER
- added R? (x4): R_US, ~, symbol R_US
- added X?: 12MHz, ~, symbol CRYSTAL
- gave numbers to parts that had none: 1
Connections:
- net labels added: +1.8V, CTS2, RTS2, RxD1, RxD2, TxD1, TxD2
- wire segments 36 -> 130
Other:
- moved on the sheet: C?, R?, U?
