File: src/PCB/Main Board/obd.sch (KiCad schematic (older format))
At the start: 0 parts

Commit message: Updated PCB projects.
Parts:
- added C? (x2): 27pF, ~, symbol C_SMALL
- added C?: 10uF, ~, symbol CP1
- added C? (x2): 1uF, ~, symbol C_SMALL
- added D?: OBD_RX, ~, symbol LED
- added D?: OBD_TX, ~, symbol LED
- added R? (x2): R_US, ~, symbol R_US
- added U?: STN1110, ~, symbol STN1110
- added X?: 16Mhz, ~, symbol CRYSTAL
Connections:
- new net: C?.1, U?.10 (OSC2), X?.2
- new net: C?.1, U?.20 (VCAP)
- new net: R?.1, U?.21 (~OBD_TX_LED~/~RST_NVM)
- new net: R?.1, U?.22 (~OBD_RX_LED~/~INT)
- new net: C?.1, U?.8 (VSS), X?.1
- new net: D?.1 (A), R?.2 (x2)
- new net +3.3V: C?.1, C?.1, D?.2 (K), D?.2 (K), U?.13 (VDD), U?.28 (AVDD)
- new net GND: C?.2, C?.2, C?.2, C?.2, C?.2, U?.19 (VSS), U?.27 (AVSS), U?.9 (OSC1)
- new net UART_RX: U?.17 (UART_TX)
- new net UART_TX: U?.16 (UART_RX)
